File: Print/Vorlage ATmega644PA.brd (EAGLE design)
At the start: 160 x 100 mm, 108 parts, among them IC1 ATmega644PA, IC2 LP2985-XXDBVR, IC3 74AC165D, IC4 ATTINY24/44/84-SSU, Q1 16MHz, Q2 32.768kHz, X1 

Commit message: print fertig
Parts:
- removed 3.3V, VCC: 3.3V, solpad:LSP11
- removed C10: 100uF, rcl2:UD-6,3X5,8_NICHICON
- removed C13, C18: 1uF, rcl:C0805
- removed C14, C17: 100nF, rcl:C0805
- removed C15: 12pF, rcl:C0805
- removed C16: 12pF, rcl:C0805K
- removed C6: 100nF, rcl:C1206
- removed F2: 500mA, fuse:F1206
- removed H1, H3, H5, H7: rot, led:CHIPLED_1206
- removed H2, H4, H6, H8: blau, led:CHIPLED_1206
- removed IC2: LP2985-XXDBVR, SmartPrj:SOT23-DBV
- removed IC3: 74AC165D, 74xx-eu:SO16
- removed LCD-POWER, LED-POWER: (no value), jumper:JP1
- removed LCD1: EADIP203-4_SMD, display-lcd:EADIP203-4SMD
- removed LCD_POTI: 2k5, pot:3223G
- removed PORT_A, PORT_A2, PORT_D: (no value), jumper:JP5Q
- removed Q2: 32.768kHz, crystal:TC38H
- removed R12: 1k, rcl:R1206
- removed R13: 1k, rcl:R0805
- removed R14, R16: 2k, rcl:R0805
- removed R15: 150R, rcl:R1206
- removed R23, R24, R35, R38, R39, R40, R41, R43: 100k, rcl:R0805
- removed R25, R26, R27, R28, R29, R30, R31, R32: 150R, rcl:R0805
- removed RS232_BT: (no value), jumper:JP3Q
- removed S3, S4: (no value), SmartPrj:TS42_4PAD
- removed S5: 219-08, switch-dil:CTS-219-08
- removed U$1: MICRO-USB, con-molex-usb:47589-0001
- removed UART_ROBO: (no value), jumper:JP2
- removed V1, V2, V3, V4, V5, V6, V7, V8: PMV20EN, transistor-fet-mit-BSS138:SOT23
- added JP1, JP2, JP3, JP4: (no value), jumper:JP2Q
- added PIEZO-POWER1, PIEZO-POWER2: (no value), jumper:JP1
- added R17: 150R, rcl:R0805
- added R21: 1k, rcl:R1206
- added U$2: DCDC, untitled:1X2,3_2.54MM
- added UART_ROBO2: (no value), jumper:JP2
- added V12: PMV20EN, transistor-fet-mit-BSS138:SOT23
- added X3: 87758-3416, con-molex:87758-3416
- C2, C4: device rcl:C1206 -> rcl:C0805
- R10, R9: value 1k -> 150R
- R11: device rcl:R0805 -> rcl:R1206
- R6, R7: value 100k -> 150R
- X1: value (none) -> (none); device con_sirius:MKDSN1,5/2-5,08 -> con-berg:PN87520
- moved C5 189.7 mm to (53.0, 12.4), flipped to the bottom, turned to 270 degrees
- moved R2 180.6 mm to (64.1, 6.86), flipped to the bottom
- moved C3 179.1 mm to (53.0, 23.0), flipped to the bottom, turned to 270 degrees
- moved R1 171.8 mm to (68.8, 22.6), flipped to the bottom
- moved C4 165.0 mm to (37.5, 14.7), turned to 180 degrees
- moved C2 159.7 mm to (41.9, 20.0), turned to 180 degrees
- moved R9 155.6 mm to (39.5, 30.6), flipped to the bottom, turned to 90 degrees
- moved R5 154.9 mm to (63.2, 21.5), flipped to the bottom
- moved UART_ROBO1 151.4 mm to (77.0, 6.99), turned to 90 degrees
- moved R11 147.7 mm to (69.2, 36.1), flipped to the bottom
- moved R8 144.1 mm to (33.3, 34.1), turned to 270 degrees
- moved Q1 143.7 mm to (47.2, 18.7), turned to 90 degrees
- moved IC1 142.1 mm to (38.9, 20.3), flipped to the bottom
- moved R4 138.7 mm to (64.1, 9.02), flipped to the bottom
- moved D2 135.2 mm to (18.7, 38.2), flipped to the bottom, turned to 90 degrees
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Connections:
- removed net 3.3V: 3.3V.MP, C14.1, C18.1, IC2.5, LCD1.2, LCD_POTI.2, LCD_POTI.3
- removed net N$12: LCD-POWER.2, R15.2
- removed net N$13: H1.A, H2.A, H3.A, H4.A, H5.A, H6.A, H7.A, H8.A, LED-POWER.2
- removed net N$17: IC3.6, R43.1, S5.16
- removed net N$18: IC3.5, R23.1, S5.15
- removed net N$23: R10.1, R7.1, S4.3, S4.4
- removed net N$24: R6.1, R9.1, S3.3, S3.4
- removed net N$25: H4.C, R28.2
- removed net N$26: H3.C, R27.2
- removed net N$30: R27.1, V3.3
- removed net N$31: IC3.4, R24.1, S5.14
- removed net N$32: R28.1, V4.3
- removed net N$34: LCD1.3, LCD_POTI.1
- removed net N$39: LCD1.6, R11.1, R14.2
- removed net N$4: U$3.REMOTE, UART_ROBO1.2
- removed net N$40: LCD1.5, R13.1, R16.2
- removed net N$42: H6.C, R30.2
- removed net N$43: H5.C, R29.2
- removed net N$44: R29.1, V5.3
- removed net N$45: R30.1, V6.3
- removed net N$48: H8.C, R32.2
- removed net N$49: H7.C, R31.2
- removed net N$50: R31.1, V7.3
- removed net N$51: R32.1, V8.3
- removed net N$59: IC3.3, R35.1, S5.13
- removed net N$61: IC3.14, R38.1, S5.12
- removed net N$62: IC3.13, R39.1, S5.11
- removed net N$63: IC3.12, R40.1, S5.10
- removed net N$64: IC3.11, R41.1, S5.9
- removed net N$66: IC3.9, R12.1
- removed net N$70: C17.1, IC2.4
- removed net N$8: R26.1, V2.3
- removed net N$95: LCD1.17, R15.1
- removed net PB0_: IC4.2, PORT_A2.2
- removed net PB1_: IC4.3, PORT_A2.4
- removed net PB2_: IC4.5, PORT_A2.6
- removed net PB3_: IC4.4, PORT_A2.8
- removed net V_AKKU: F1.1, X1.2.1, X1.2.2
- new net N$1: X3.1
- new net N$10: X3.3
- new net N$11: X3.5
- new net N$19: X3.7
- new net N$2: X3.2
- new net N$20: X3.9
- new net N$29: X3.11
- new net N$33: X3.13
- new net N$41: X3.15
- new net N$46: PIEZO-POWER2.2, R21.2, V12.3
- new net N$47: X3.19
- new net N$52: X3.21
- new net N$53: X3.23
- new net N$54: X3.25
- new net N$55: X3.27
- new net N$56: X3.29
- new net N$57: X3.31
- new net N$58: X3.32
- new net N$65: X3.30
- new net N$67: X3.28
- new net N$68: X3.26
- new net N$69: X3.24
- new net N$71: X3.22
- new net N$73: X3.18
- new net N$74: X3.16
- new net N$76: X3.14
- new net N$77: X3.12
- new net N$78: X3.10
- new net N$79: X3.8
- new net N$80: X3.6
- new net N$82: X3.34
- new net N$83: X3.33
- new net N$85: R17.2, U$2.TRIM
- new net PD8: PIEZO-POWER1.2, R11.1, V12.1
- new net RX: JP1.3, JTAG.6, X3.17
- new net TX: JP1.2, JTAG.8, X3.20
- net +12V: now also F1.1, J1.3, JP3.1, JP3.3, U$2.V_IN; no longer UART_ROBO1.3
- net +5V: now also U$2.V_OUT, X1.1; no longer C13.1, C2.1, C4.1, C7.1, IC1.17, IC1.38, IC1.5, IC2.1, IC2.3, IC4.1, JTAG.4, R5.2, S5.1, S5.2, S5.3, S5.4, S5.5, S5.6, S5.7, S5.8
- net DGND: now also R17.1, R18.1, U$2.GND, U$3.GND; no longer C13.2, C17.2, C18.2, IC2.2, IC3.10, IC3.15, JTAG.10, JTAG.2, R23.2, R24.2, R35.2, R38.2, R39.2, R40.2, R41.2, R43.2
- net GND: now also J1.1, J1.2, JP3.2, JP3.4, JTAG.10, JTAG.2, R11.2, UART_ROBO2.1, UART_ROBO2.2, UART_ROBO2.3, V12.2, X1.4, X3.4; no longer C10.-, C14.2, C15.2, C16.2, C6.2, IC3.8, LCD1.1, LCD1.18, LCD1.4, PORT_A.1, PORT_A.10, PORT_D.1, PORT_D.10, R14.1, R16.1, R18.1, R6.2, R7.2, RS232_BT.5, RS232_BT.6, U$1.5, U$1.CASING1, U$1.CASING2, U$1.CASING3, U$1.CASING4, U$1.CASING5, U$1.CASING6, U$1.CASING7, U$1.CASING8, U$3.GND, UART_ROBO.1, UART_ROBO1.1, V1.2, V2.2, V3.2, V4.2, V5.2, V6.2, V7.2, V8.2, X1.1.1, X1.1.2
- net N$14: now also JP2.3; no longer RS232_BT.2
- net N$15: now also JP2.1; no longer RS232_BT.4
- net N$3: now also IC4.4, R10.2; no longer F2.1, U$1.1
- net N$5: now also IC4.5, R9.2; no longer H2.C, R26.2
- net N$6: now also IC4.3, R7.2; no longer H1.C, R25.2
- net N$7: now also IC4.2, R6.2; no longer R25.1, V1.3
- net PA0: now also R6.1; no longer PORT_A.2, PORT_A2.1
- net PA1: now also R7.1; no longer PORT_A.3, PORT_A2.3
- net PA2: now also R9.1; no longer PORT_A.4, PORT_A2.5
- net PA3: now also R10.1; no longer PORT_A.5, PORT_A2.7
- net PA4: no longer PORT_A.6
- net PA5: no longer IC3.1, PORT_A.7
- net PA6: no longer IC3.2, PORT_A.8
- net PA7: no longer PORT_A.9, R12.2
- net PB0: no longer V8.1
- net PB1: no longer V7.1
- net PB2: no longer R9.2, V6.1
- net PB3: no longer R10.2, V5.1
- net PB4: no longer V4.1
- net PB5: no longer V3.1
- net PB6: no longer V2.1
- net PB7: no longer V1.1
- net PC0: no longer R13.2
- net PC1: no longer R11.2
- net PC6: no longer C16.1, Q2.2
- net PC7: no longer C15.1, Q2.1
- net PD0: now also JP2.2; no longer PORT_D.2, RS232_BT.3
- net PD1: now also JP2.4; no longer PORT_D.3, RS232_BT.1
- net PD2: now also JP1.1; no longer PORT_D.4, UART_ROBO.2
- net PD3: now also JP1.4, PIEZO-POWER1.1; no longer PORT_D.5, UART_ROBO.3
- net PD4: now also JP4.1; no longer PORT_D.6
- net PD5: now also JP4.2; no longer PORT_D.7
- net PD6: now also JP4.3; no longer PORT_D.8
- net PD7: now also JP4.4; no longer PORT_D.9
- net VCC: now also C2.1, C4.1, C7.1, IC1.17, IC1.38, IC1.5, IC4.1, JTAG.4, PIEZO-POWER2.1, R21.1, R5.2, UART_ROBO1.1, UART_ROBO1.2, UART_ROBO1.3; no longer C10.+, C6.1, F2.2, IC3.16, LCD-POWER.1, LED-POWER.1, S3.1, S3.2, S4.1, S4.2, VCC.MP
Routing:
- net VCC: track 0.00 -> 221.6 mm, vias 0 -> 3
- net DGND: track 0.00 -> 106.2 mm, vias 0 -> 4
- net RX: track 0.00 -> 50.3 mm
- net PB1: track 0.00 -> 40.8 mm
- net +5V: track 0.00 -> 40.6 mm
- net PA7_: track 0.00 -> 36.7 mm, vias 0 -> 1
- net PD8: track 0.00 -> 36.2 mm, vias 0 -> 1
- net PB0: track 0.00 -> 34.4 mm, vias 0 -> 2
- net PA6_: track 0.00 -> 33.9 mm, vias 0 -> 1
- net +12V: track 0.00 -> 33.1 mm
- net RESET: track 0.00 -> 33.1 mm, vias 0 -> 2
- net PA3_: track 0.00 -> 33.0 mm, vias 0 -> 1
- net PA5_: track 0.00 -> 32.9 mm, vias 0 -> 1
- net PA1_: track 0.00 -> 32.1 mm, vias 0 -> 1
- net PC4: track 0.00 -> 30.4 mm, vias 0 -> 1
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- added copper zone on layer 1, net GND
- added copper zone on layer 16, net GND
Other:
- board size 160 x 100 mm -> 80 x 45 mm

Commit message: asd
Routing:
- net GND: track 13.7 -> 8.21 mm
- added copper zone on layer 15, net +5V

Commit message: sf
Parts:
- removed J1: (no value), con-jack:SPC4077
- added U$1: BUCHSE, untitled:BUCHSE
- moved PIEZO-POWER2 10.0 mm to (77.5, 30.9)
- moved R21 4.22 mm to (73.4, 30.5)
- moved X1 0.89 mm to (5.80, 9.33)
- moved JP3 0.63 mm to (16.8, 24.8)
- moved R3 0.40 mm to (69.2, 20.4)
Connections:
- net +12V: now also U$1.3, U$1.3.1; no longer J1.3
- net +5V: now also UART_ROBO1.1, UART_ROBO1.2, UART_ROBO1.3
- net DGND: now also JP3.2, JP3.4, U$1.1, U$1.2, UART_ROBO2.1, UART_ROBO2.2, UART_ROBO2.3, X1.4; no longer IC4.14
- net GND: now also IC4.14; no longer J1.1, J1.2, JP3.2, JP3.4, UART_ROBO2.1, UART_ROBO2.2, UART_ROBO2.3, X1.4
- net VCC: no longer UART_ROBO1.1, UART_ROBO1.2, UART_ROBO1.3
Routing:
- net DGND: track 106.1 -> 81.1 mm
- net VCC: track 221.6 -> 199.7 mm, vias 3 -> 4
- net N$46: track 23.4 -> 10.6 mm, vias 1 -> 0
- net +12V: track 33.1 -> 36.3 mm
- net +5V: track 40.6 -> 37.6 mm
- net N$22: track 13.0 -> 15.1 mm
- net PA5_: track 32.9 -> 34.2 mm
- net N$85: track 4.30 -> 3.44 mm
- net N$16: track 4.37 -> 3.65 mm
- net PD3: track 18.7 -> 18.0 mm
- net PC5: track 20.6 -> 20.0 mm
- net N$7: track 4.03 -> 4.62 mm
- added copper zone on layer 2, net DGND
