File: Print/Vorlage ATmega644PA.brd (EAGLE design)
At the start: 84 x 45 mm, 58 parts, among them IC1 ATmega644PA, IC4 ATTINY24/44/84-SSU, Q1 16MHz

Commit message: asd
Changed lines of the file:
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@@
 <wire x1="43.2562" y1="17.1704" x2="43.0911" y2="17.3355" width="0.508" layer="16"/>
 <wire x1="44.577" y1="19.3167" x2="44.67" y2="19.303" width="0.508" layer="16"/>
-<wire x1="17.5006" y1="33.8455" x2="17.5006" y2="33.6804" width="0.508" layer="1"/>
-<wire x1="17.6657" y1="34.0106" x2="17.5006" y2="33.8455" width="0.508" layer="1"/>
 <wire x1="16.1798" y1="31.0388" x2="16.05" y2="31" width="0.508" layer="1"/>
-<wire x1="17.6657" y1="34.0106" x2="17.74" y2="34" width="0.508" layer="1"/>
 <wire x1="17.8308" y1="37.4777" x2="17.719" y2="37.592" width="0.508" layer="1"/>
 <wire x1="8.4201" y1="18.9865" x2="8.489" y2="19.173" width="0.508" layer="1"/>
@@
 <wire x1="38.1" y1="13.473" x2="38.1" y2="12.1793" width="0.508" layer="16"/>
 <wire x1="38.1" y1="12.1793" x2="37.973" y2="12.0523" width="0.508" layer="16"/>
-<wire x1="43.2562" y1="19.3167" x2="38.87" y2="25.103" width="0" layer="19" extent="16-16"/>
-<wire x1="38.07" y1="13.503" x2="43.0911" y2="17.3355" width="0" layer="19" extent="16-16"/>
-<wire x1="33.07" y1="19.303" x2="38.07" y2="13.503" width="0" layer="19" extent="16-16"/>
-<wire x1="44.46" y1="3.5" x2="37.973" y2="12.0523" width="0" layer="19" extent="1-1"/>
-<wire x1="47" y1="3.5" x2="44.46" y2="3.5" width="0" layer="19" extent="1-1"/>
-<wire x1="49.54" y1="3.5" x2="47" y2="3.5" width="0" layer="19" extent="1-1"/>
-<wire x1="17.034" y1="10.495" x2="31.6992" y2="19.1516" width="0" layer="19" extent="16-16"/>
-<wire x1="8.512" y1="5.832" x2="12.619" y2="10.495" width="0" layer="19" extent="1-1"/>
-<wire x1="16.05" y1="31" x2="7.731" y2="21.987" width="0" layer="19" extent="1-1"/>
 </signal>
 <signal name="N$27">
@@
 <contactref element="PORT_A1" pad="1"/>
 <wire x1="64.7192" y1="36.4871" x2="59.436" y2="36.4871" width="0.508" layer="16"/>
-<wire x1="77.7621" y1="23.4442" x2="64.7192" y2="36.4871" width="0.508" layer="1"/>
-<wire x1="79.4258" y1="23.4442" x2="77.7621" y2="23.4442" width="0.508" layer="1"/>
+<wire x1="77.6351" y1="23.5712" x2="64.7192" y2="36.4871" width="0.508" layer="1"/>
+<wire x1="79.5528" y1="23.5712" x2="77.6351" y2="23.5712" width="0.508" layer="1"/>
 <wire x1="80.881" y1="24.978" x2="80.881" y2="24.8994" width="0.508" layer="1"/>
-<wire x1="80.881" y1="24.8994" x2="79.4258" y2="23.4442" width="0.508" layer="1"/>
+<wire x1="80.881" y1="24.8994" x2="79.5528" y2="23.5712" width="0.508" layer="1"/>
 <wire x1="59.436" y1="36.4871" x2="59.4281" y2="36.4812" width="0.508" layer="16"/>
 <via x="64.7192" y="36.4871" extent="1-16" drill="0.508"/>
@@
 <contactref element="IC4" pad="10"/>
 <contactref element="PORT_A1" pad="3"/>
-<wire x1="64.8843" y1="39.1287" x2="59.436" y2="39.1287" width="0.508" layer="16"/>
+<wire x1="64.8843" y1="39.1287" x2="64.7573" y2="39.0017" width="0.508" layer="16"/>
+<wire x1="64.7573" y1="39.0017" x2="59.4476" y2="39.0017" width="0.508" layer="16"/>
+<wire x1="59.4281" y1="39.0212" x2="59.4476" y2="39.0017" width="0.508" layer="16"/>
 <wire x1="65.2145" y1="39.1287" x2="64.8843" y2="39.1287" width="0.508" layer="1"/>
-<wire x1="68.1863" y1="36.1569" x2="65.2145" y2="39.1287" width="0.508" layer="1"/>
-<wire x1="70.1675" y1="36.1569" x2="68.1863" y2="36.1569" width="0.508" layer="1"/>
-<wire x1="77.597" y1="28.7274" x2="70.1675" y2="36.1569" width="0.508" layer="1"/>
+<wire x1="66.7893" y1="37.5539" x2="65.2145" y2="39.1287" width="0.508" layer="1"/>
+<wire x1="68.7705" y1="37.5539" x2="66.7893" y2="37.5539" width="0.508" layer="1"/>
+<wire x1="77.597" y1="28.7274" x2="68.7705" y2="37.5539" width="0.508" layer="1"/>
 <wire x1="79.248" y1="28.7274" x2="77.597" y2="28.7274" width="0.508" layer="1"/>
 <wire x1="80.4037" y1="27.5717" x2="79.248" y2="28.7274" width="0.508" layer="1"/>
 <wire x1="80.7339" y1="27.5717" x2="80.4037" y2="27.5717" width="0.508" layer="1"/>
-<wire x1="59.436" y1="39.1287" x2="59.4281" y2="39.0212" width="0.508" layer="16"/>
 <wire x1="80.7339" y1="27.5717" x2="80.881" y2="27.518" width="0.508" layer="1"/>
 <via x="64.8843" y="39.1287" extent="1-16" drill="0.508"/>
@@
 <contactref element="PORT_A1" pad="6"/>
 <wire x1="65.0494" y1="40.2844" x2="59.436" y2="40.2844" width="0.508" layer="16"/>
-<wire x1="68.5165" y1="36.8173" x2="65.0494" y2="40.2844" width="0.508" layer="1"/>
-<wire x1="70.993" y1="36.8173" x2="68.5165" y2="36.8173" width="0.508" layer="1"/>
-<wire x1="77.7621" y1="30.0482" x2="70.993" y2="36.8173" width="0.508" layer="1"/>
+<wire x1="66.7385" y1="38.5953" x2="65.0494" y2="40.2844" width="0.508" layer="1"/>
+<wire x1="69.215" y1="38.5953" x2="66.7385" y2="38.5953" width="0.508" layer="1"/>
+<wire x1="77.7621" y1="30.0482" x2="69.215" y2="38.5953" width="0.508" layer="1"/>
 <wire x1="78.2574" y1="30.0482" x2="77.7621" y2="30.0482" width="0.508" layer="1"/>
 <wire x1="59.436" y1="40.2844" x2="59.4281" y2="40.2912" width="0.508" layer="16"/>
@@
 <wire x1="52.9971" y1="41.6052" x2="54.1528" y2="41.6052" width="0.508" layer="16"/>
 <wire x1="52.5018" y1="41.1099" x2="52.9971" y2="41.6052" width="0.508" layer="16"/>
-<wire x1="64.5541" y1="41.1099" x2="52.5018" y2="41.1099" width="0.508" layer="1"/>
-<wire x1="64.7192" y1="41.275" x2="64.5541" y2="41.1099" width="0.508" layer="1"/>
-<wire x1="69.1769" y1="41.275" x2="64.7192" y2="41.275" width="0.508" layer="1"/>
-<wire x1="77.7621" y1="32.6898" x2="69.1769" y2="41.275" width="0.508" layer="1"/>
+<wire x1="69.3039" y1="41.148" x2="52.5399" y2="41.148" width="0.508" layer="1"/>
+<wire x1="52.5399" y1="41.148" x2="52.5018" y2="41.1099" width="0.508" layer="1"/>
+<wire x1="77.7621" y1="32.6898" x2="69.3039" y2="41.148" width="0.508" layer="1"/>
 <wire x1="77.7720875" y1="32.6898" x2="77.7621" y2="32.6898" width="0.508" layer="1"/>
 <wire x1="54.1528" y1="41.6052" x2="54.2211" y2="41.5612" width="0.508" layer="16"/>

Commit message: print fertig
Parts:
- removed JP2: (no value), jumper:JP2Q
- added PIEZO-POWER6: (no value), jumper:JP1
- added X2: 87758-0616, con-molex:87758-0616
- R17, R18: value 150R -> 1k472
- moved X1 72.7 mm to (78.5, 9.97), turned to 90 degrees
- moved JTAG 25.6 mm to (4.65, 27.6), turned to 90 degrees
- moved PIEZO-POWER1 18.3 mm to (77.5, 21.0)
- moved U$1 16.4 mm to (14.0, 8.79)
- moved R3 15.6 mm to (64.0, 19.5), turned to 90 degrees
- moved R21 15.5 mm to (77.1, 25.5)
- moved PIEZO-POWER2 15.5 mm to (81.5, 25.5)
- moved R1 15.4 mm to (61.9, 19.5), turned to 90 degrees
- moved S2 15.2 mm to (70.0, 19.5), turned to 90 degrees
- moved R2 14.6 mm to (68.5, 19.6)
- moved R4 14.6 mm to (70.6, 19.5)
- moved S1 14.5 mm to (63.6, 19.5), turned to 90 degrees
- moved L1 13.3 mm to (42.0, 19.6), turned to 180 degrees
- moved V12 12.6 mm to (73.5, 29.4), turned to 180 degrees
- moved JP3 12.3 mm to (27.9, 13.7)
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Connections:
- net N$5 renamed PB2_
- net N$6 renamed PB1_
- net N$7 renamed PB0_
- removed net N$14: JP2.3, RN1.5
- removed net N$15: JP2.1, RN1.4
- removed net N$3: IC4.4, R10.2
- new net PB3_: IC4.4, R10.2, X2.5
- net GND: now also X2.6
- net PA4_: now also X2.3
- net PA5_: now also X2.1
- net PA6_: now also X2.4
- net PD0: now also PIEZO-POWER6.2, RN1.4; no longer JP2.2
- net PD1: now also PIEZO-POWER6.1, RN1.5; no longer JP2.4
- net VCC: now also X2.2
Routing:
- net PD0: track 11.9 -> 52.5 mm, vias 0 -> 1
- net VCC: track 233.4 -> 193.7 mm
- net PC3: track 27.2 -> 58.9 mm
- net N$3: track 23.3 -> 0.00 mm
- net N$15: track 23.1 -> 0.00 mm
- net RX: track 62.0 -> 84.9 mm
- net PD8: track 37.0 -> 14.4 mm, vias 2 -> 0
- net N$14: track 20.4 -> 0.00 mm
- net PB3_: track 0.00 -> 20.3 mm
- net TX: track 59.8 -> 79.6 mm, vias 0 -> 1
- net PB0: track 41.7 -> 22.9 mm
- net N$36: track 30.1 -> 11.5 mm
- net +12V: track 49.9 -> 68.2 mm
- net PD1: track 11.4 -> 29.7 mm
- net RESET: track 36.8 -> 19.6 mm, vias 1 -> 2
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Other:
- board text added: "C:/Users/Jan Spuler/OneDrive - MSW-Winterthur/Desktop/bt.bmp"
- board text added: "D1 0"
- board text added: "piezo"
- board text added: "pwr"

Commit message: asd
Parts:
- removed GND: 3.3V, solpad:LSP11
- removed PIEZO-POWER6: (no value), jumper:JP1
- removed X2: 87758-0616, con-molex:87758-0616
- added JP2: (no value), jumper:JP3Q
- added R12, R13: 1k, rcl:R0805
- added RX, TX: Gruen, led:CHIPLED_1206
- added V1, V2: PMV20EN, transistor-fet-mit-BSS138:SOT23
Connections:
- new net N$2: TX.C, V2.3
- new net N$3: RX.C, V1.3
- new net N$4: R13.1, TX.A
- new net N$5: R12.1, RX.A
- net GND: now also JP2.1, U$4.31, V1.2, V2.2; no longer GND.MP, X2.6
- net PA4_: now also JP2.4; no longer X2.3
- net PA5_: now also JP2.6; no longer X2.1
- net PA6_: now also JP2.3; no longer X2.4
- net PB3_: now also JP2.2; no longer X2.5
- net PD0: no longer PIEZO-POWER6.2
- net PD1: now also V2.1; no longer PIEZO-POWER6.1
- net PD3: now also V1.1
- net RX: now also U$4.18; no longer U$4.17
- net TX: now also U$4.19; no longer U$4.20
- net VCC: now also JP2.5, R12.2, R13.2; no longer X2.2
Routing:
- net PD3: track 41.5 -> 64.1 mm, vias 0 -> 2
- net VCC: track 193.7 -> 204.4 mm
- net N$5: track 0.00 -> 7.55 mm
- net N$4: track 0.00 -> 7.51 mm
- net PD0: track 52.5 -> 46.1 mm
- net N$3: track 0.00 -> 6.35 mm, vias 0 -> 1
- net PA5_: track 40.5 -> 36.7 mm
- net N$2: track 0.00 -> 3.59 mm, vias 0 -> 1
- net PA4_: track 29.3 -> 31.3 mm, vias 1 -> 0
- net TX: track 79.6 -> 77.8 mm
- net PA6_: track 39.5 -> 40.9 mm, vias 0 -> 1
- net DGND: track 38.9 -> 38.0 mm
- net PB3_: track 20.3 -> 20.5 mm, vias 0 -> 1
- net PD1: track 29.7 -> 29.6 mm, vias 1 -> 2
Other:
- board text removed: "D1 0"
