File: Print/Vorlage ATmega644PA.sch (EAGLE design)
At the start: 103 parts, among them IC1 ATmega644PA, IC2 LP2985-XXDBVR, IC3 74AC165D, Q1 16MHz, Q2 32.768kHz, X1 

Commit message: ll
Parts:
- removed R17: 240R, rcl:R-EU_R0805
- removed SENSOR/SERVO: (no value), jumper:JP2E
- removed U$2: DC-DC_WANDLER, untitled:DC-DC_WANDLER
- added IC4: ATTINY24/44/84-SSU, attiny24_44_84:ATTINY24/44/84-SSU
- added PORT_A1, PORT_A2: (no value), jumper:JP5Q
- added R18: 150R, rcl:R-EU_R0805
- added U$3: DCDC, untitled:DCDC
- added UART_ROBO, UART_ROBO1: (no value), jumper:JP2E
Connections:
- removed net N$1: U$2.L
- removed net N$10: U$2.VOUT
- removed net N$11: R17.2, U$2.TRIM
- removed net N$2: U$2.N
- new net +12V: U$3.VIN, UART_ROBO1.3
- new net N$16: R18.2, U$3.TRIM
- new net N$27: PORT_A1.9
- new net N$28: PORT_A1.10
- new net N$4: U$3.REMOTE, UART_ROBO1.2
- new net PA0_: IC4.(PCINT0/AREF/ADC0)PA0, PORT_A1.2
- new net PA1_: IC4.(PCINT1/AIN0/ADC1)PA1, PORT_A1.1
- new net PA2_: IC4.(PCINT2/AIN1/ADC2)PA2, PORT_A1.4
- new net PA3_: IC4.(PCINT3/T0/ADC3)PA3, PORT_A1.3
- new net PA4_: IC4.(PCINT4/T1/SCL/USCK/ADC4)PA4, PORT_A1.6
- new net PA5_: IC4.(PCINT5/OC1B/MISO/DO/ADC5)PA5, PORT_A1.5
- new net PA6_: IC4.(PCINT6/OC1A/SDA/MOSI/ADC6)PA6, PORT_A1.8
- new net PA7_: IC4.(PCINT7/ICP/OC0B/ADC7)PA7, PORT_A1.7
- new net PB0_: IC4.(PCINT8/XTAL1/CLKI)PB0, PORT_A2.2
- new net PB1_: IC4.(PCINT9/XTAL2)PB1, PORT_A2.4
- new net PB2_: IC4.(PCINT10/INT0/OC0A/CKOUT)PB2, PORT_A2.6
- new net PB3_: IC4.(PCINT11/RESET/DW)PB3, PORT_A2.8
- net +5V: now also IC4.VCC, U$3.VOUT
- net DGND: now also IC4.GND
- net GND: now also R18.1, U$3.GND, UART_ROBO.1, UART_ROBO1.1; no longer R17.1, SENSOR/SERVO.1, U$2.GND
- net PA0: now also PORT_A2.1
- net PA1: now also PORT_A2.3
- net PA2: now also PORT_A2.5
- net PA3: now also PORT_A2.7; no longer SENSOR/SERVO.3
- net PB0: now also V8.G
- net PB1: now also V7.G
- net PB2: now also V6.G
- net PB3: now also V5.G
- net PB4: now also V4.G
- net PB5: now also V3.G
- net PB6: now also V2.G
- net PB7: now also V1.G
- net PD2: now also UART_ROBO.2
- net PD3: now also UART_ROBO.3
- net VCC: no longer SENSOR/SERVO.2
Other:
- note added: "RX"
- note added: "RX_ROBO"
- note added: "TX"
- note added: "TX_ROBO"
- note added: "com mit tiny"
- note removed: "1. Juli 2015"
- note removed: "2xLED Weiss"
- note removed: "Enable H-Brücke Left"
- note removed: "Enable H-Brücke Right"
- note removed: "GND"
- note removed: "Joystick X-Achse"
- note removed: "Joystick Y-Achse"
- note removed: "Lichtsensor"
- note removed: "Mein erstes Board"
- note removed: "RGB Blau"
- note removed: "RGB Gruen"
- note removed: "RGB Rot"
- note removed: "Sensor A"
- note removed: "Sensor/Servo"
- note removed: "Sig"
- note removed: "Vcc"

Commit message: asd
Parts:
- added J1: (no value), con-jack:JACK-PLUG0
Changed lines of the file:
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@@
 <part name="GND13" library="supply1" deviceset="GND" device=""/>
 <part name="P+3" library="supply1" library_urn="urn:adsk.eagle:library:371" deviceset="+12V" device=""/>
+<part name="J1" library="con-jack" library_urn="urn:adsk.eagle:library:154" deviceset="JACK-PLUG" device="0" package3d_urn="urn:adsk.eagle:package:7492/1"/>
 </parts>
 <sheets>
@@
 <attribute name="VALUE" x="266.7" y="45.72" size="1.778" layer="96" rot="R90"/>
 </instance>
+<instance part="J1" gate="G$1" x="350.52" y="93.98" smashed="yes">
+<attribute name="NAME" x="342.9" y="99.06" size="1.778" layer="95"/>
+<attribute name="VALUE" x="342.9" y="88.9" size="1.778" layer="96"/>
+</instance>
 </instances>

Commit message: shrt
Parts:
- added X2: (no value), con-phoenix-500:MSTBV2
Connections:
- net +12V: now also J1.3, X2-2.SK
- net GND: now also J1.1, J1.2, X2-1.SK
Changed lines of the file:
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@@
 <part name="P+3" library="supply1" library_urn="urn:adsk.eagle:library:371" deviceset="+12V" device=""/>
 <part name="J1" library="con-jack" library_urn="urn:adsk.eagle:library:154" deviceset="JACK-PLUG" device="0" package3d_urn="urn:adsk.eagle:package:7492/1"/>
+<part name="P+6" library="supply1" library_urn="urn:adsk.eagle:library:371" deviceset="+12V" device=""/>
+<part name="GND1" library="supply1" deviceset="GND" device=""/>
+<part name="X2" library="con-phoenix-500" library_urn="urn:adsk.eagle:library:175" deviceset="MSTBV2" device="" package3d_urn="urn:adsk.eagle:package:9455/1"/>
 </parts>
 <sheets>
@@
 <attribute name="VALUE" x="342.9" y="88.9" size="1.778" layer="96"/>
 </instance>
+<instance part="P+6" gate="1" x="358.14" y="101.6" smashed="yes">
+<attribute name="VALUE" x="355.6" y="96.52" size="1.778" layer="96" rot="R90"/>
+</instance>
+<instance part="GND1" gate="1" x="358.14" y="86.36" smashed="yes">
+<attribute name="VALUE" x="355.6" y="83.82" size="1.778" layer="96"/>
+</instance>
+<instance part="X2" gate="-1" x="368.3" y="91.44" smashed="yes" rot="R180">
+<attribute name="NAME" x="374.904" y="90.551" size="1.778" layer="95"/>
+</instance>
+<instance part="X2" gate="-2" x="368.3" y="96.52" smashed="yes" rot="R180">
+<attribute name="VALUE" x="375.92" y="100.33" size="1.778" layer="96" rot="R180"/>
+<attribute name="NAME" x="375.158" y="95.631" size="1.778" layer="95"/>
+</instance>
 </instances>
 <busses>
@@
 <wire x1="274.32" y1="35.56" x2="271.78" y2="35.56" width="0.1524" layer="91"/>
 </segment>
+<segment>
+<pinref part="J1" gate="G$1" pin="2"/>
+<pinref part="GND1" gate="1" pin="GND"/>
+<wire x1="355.6" y1="93.98" x2="358.14" y2="93.98" width="0.1524" layer="91"/>
+<wire x1="358.14" y1="93.98" x2="358.14" y2="91.44" width="0.1524" layer="91"/>
+<pinref part="J1" gate="G$1" pin="1"/>
+<wire x1="358.14" y1="91.44" x2="358.14" y2="88.9" width="0.1524" layer="91"/>
+<wire x1="355.6" y1="91.44" x2="358.14" y2="91.44" width="0.1524" layer="91"/>
+<junction x="358.14" y="91.44"/>
+<pinref part="X2" gate="-1" pin="SK"/>
+<wire x1="360.68" y1="91.44" x2="358.14" y2="91.44" width="0.1524" layer="91"/>
+</segment>
 </net>
 <net name="VCC" class="1">
@@
 <wire x1="269.24" y1="45.72" x2="269.24" y2="48.26" width="0.1524" layer="91"/>
 </segment>
-</net>
+<segment>
+<pinref part="J1" gate="G$1" pin="3"/>
+<pinref part="P+6" gate="1" pin="+12V"/>
+<wire x1="355.6" y1="96.52" x2="358.14" y2="96.52" width="0.1524" layer="91"/>
+<wire x1="358.14" y1="96.52" x2="358.14" y2="99.06" width="0.1524" layer="91"/>
+<pinref part="X2" gate="-2" pin="SK"/>
+<wire x1="360.68" y1="96.52" x2="358.14" y2="96.52" width="0.1524" layer="91"/>
+<junction x="358.14" y="96.52"/>
+</segment>
+</net>

Commit message: print fertig
Parts:
- removed 3.3V, VCC: 3.3V, solpad:LSP11
- removed C10: 100uF, rcl2:CPOL-EUUD-6,3X8,8
- removed C13, C18: 1uF, rcl:C-EUC0805
- removed C14, C17: 100nF, rcl:C-EUC0805
- removed C15: 12pF, rcl:C-EUC0805
- removed C16: 12pF, rcl:C-EUC0805K
- removed C6: 100nF, rcl:C-EUC1206
- removed F2: 500mA, fuse:195601206
- removed H1, H3, H5, H7: rot, led:LEDCHIPLED_1206
- removed H2, H4, H6, H8: blau, led:LEDCHIPLED_1206
- removed IC2: LP2985-XXDBVR, SmartPrj:LP2985-XXDBVR
- removed IC3: 74AC165D, 74xx-eu:74AC165D
- removed LCD-POWER, LED-POWER: (no value), jumper:JP1E
- removed LCD1: EADIP203-4_SMD, display-lcd:EADIP203-4EADIP203-4SMD
- removed LCD_POTI: 2k5, pot:TRIM_EU-3223G
- removed PORT_A, PORT_A2, PORT_D: (no value), jumper:JP5Q
- removed Q2: 32.768kHz, crystal:CRYSTALTC38H
- removed R12: 1k, rcl:R-EU_R1206
- removed R13: 1k, rcl:R-EU_R0805
- removed R14, R16: 2k, rcl:R-EU_R0805
- removed R15: 150R, rcl:R-EU_R1206
- removed R23, R24, R35, R38, R39, R40, R41, R43: 100k, rcl:R-EU_R0805
- removed R25, R26, R27, R28, R29, R30, R31, R32: 150R, rcl:R-EU_R0805
- removed RS232_BT: (no value), jumper:JP3Q
- removed S3, S4: TS42_4PAD, SmartPrj:TS42_4PAD
- removed S5: 219-08, switch-dil:219-08
- removed U$1: MICRO-USB, con-molex-usb:MICRO-USB-RECEPTACLE47589-0001
- removed UART_ROBO: (no value), jumper:JP2E
- removed V1, V2, V3, V4, V5, V6, V7, V8: PMV20EN, transistor-fet-mit-BSS138:BSS138
- removed X2: (no value), con-phoenix-500:MSTBV2
- added JP1, JP2, JP3, JP4: (no value), jumper:JP2Q
- added PIEZO-POWER1, PIEZO-POWER2: (no value), jumper:JP1E
- added R17: 150R, rcl:R-EU_R0805
- added R21: 1k, rcl:R-EU_R1206
- added U$2: DCDC, untitled:DCDC
- added UART_ROBO2: (no value), jumper:JP2E
- added V12: PMV20EN, transistor-fet-mit-BSS138:BSS138
- added X3: 87758-3416, con-molex:87758-3416
- C2, C4: device rcl:C-EUC1206 -> rcl:C-EUC0805
- R10, R9: value 1k -> 150R
- R11: device rcl:R-EU_R0805 -> rcl:R-EU_R1206
- R6, R7: value 100k -> 150R
- X1: value (none) -> (none); device con_sirius:MKDSN1,5/2-5,08 -> con-berg:PN87520
Connections:
- removed net 3.3V: 3.3V.MP, C14.1, C18.1, IC2.OUT, LCD1.VCC, LCD_POTI.E, LCD_POTI.S
- removed net N$12: LCD-POWER.2, R15.2
- removed net N$13: H1.A, H2.A, H3.A, H4.A, H5.A, H6.A, H7.A, H8.A, LED-POWER.2
- removed net N$17: IC3A.H, R43.1, S5.16
- removed net N$18: IC3A.G, R23.1, S5.15
- removed net N$23: R10.1, R7.1, S4.3, S4.4
- removed net N$24: R6.1, R9.1, S3.3, S3.4
- removed net N$25: H4.C, R28.2
- removed net N$26: H3.C, R27.2
- removed net N$30: R27.1, V3.D
- removed net N$31: IC3A.F, R24.1, S5.14
- removed net N$32: R28.1, V4.D
- removed net N$34: LCD1.CONTR, LCD_POTI.A
- removed net N$39: LCD1.E(SCLK), R11.1, R14.2
- removed net N$4: U$3.REMOTE, UART_ROBO1.2
- removed net N$40: LCD1.R/W(SID), R13.1, R16.2
- removed net N$42: H6.C, R30.2
- removed net N$43: H5.C, R29.2
- removed net N$44: R29.1, V5.D
- removed net N$45: R30.1, V6.D
- removed net N$48: H8.C, R32.2
- removed net N$49: H7.C, R31.2
- removed net N$50: R31.1, V7.D
- removed net N$51: R32.1, V8.D
- removed net N$59: IC3A.E, R35.1, S5.13
- removed net N$61: IC3A.D, R38.1, S5.12
- removed net N$62: IC3A.C, R39.1, S5.11
- removed net N$63: IC3A.B, R40.1, S5.10
- removed net N$64: IC3A.A, R41.1, S5.9
- removed net N$66: IC3A.QH, R12.1
- removed net N$70: C17.1, IC2.NC/FB
- removed net N$8: R26.1, V2.D
- removed net N$95: LCD1.LED+, R15.1
- removed net PB0_: IC4.(PCINT8/XTAL1/CLKI)PB0, PORT_A2.2
- removed net PB1_: IC4.(PCINT9/XTAL2)PB1, PORT_A2.4
- removed net PB2_: IC4.(PCINT10/INT0/OC0A/CKOUT)PB2, PORT_A2.6
- removed net PB3_: IC4.(PCINT11/RESET/DW)PB3, PORT_A2.8
- removed net V_AKKU: F1.1, X1-V+.KL
- new net N$1: X3-1.S
- new net N$10: X3-3.S
- new net N$11: X3-5.S
- new net N$19: X3-7.S
- new net N$2: X3-2.S
- new net N$20: X3-9.S
- new net N$29: X3-11.S
- new net N$33: X3-13.S
- new net N$41: X3-15.S
- new net N$46: PIEZO-POWER2.2, R21.2, V12.D
- new net N$47: X3-19.S
- new net N$52: X3-21.S
- new net N$53: X3-23.S
- new net N$54: X3-25.S
- new net N$55: X3-27.S
- new net N$56: X3-29.S
- new net N$57: X3-31.S
- new net N$58: X3-32.S
- new net N$65: X3-30.S
- new net N$67: X3-28.S
- new net N$68: X3-26.S
- new net N$69: X3-24.S
- new net N$71: X3-22.S
- new net N$73: X3-18.S
- new net N$74: X3-16.S
- new net N$76: X3-14.S
- new net N$77: X3-12.S
- new net N$78: X3-10.S
- new net N$79: X3-8.S
- new net N$80: X3-6.S
- new net N$82: X3-34.S
- new net N$83: X3-33.S
- new net N$85: R17.2, U$2.TRIM
- new net PD8: PIEZO-POWER1.2, R11.1, V12.G
- new net RX: JP1.3, JTAG.6, X3-17.S
- new net TX: JP1.2, JTAG.8, X3-20.S
- net +12V: now also F1.1, JP3.1, JP3.3, U$2.VIN; no longer UART_ROBO1.3, X2-2.SK
- net +5V: now also U$2.VOUT, X1.1; no longer C13.1, C2.1, C4.1, C7.1, IC1.VCC, IC1.VCC@1, IC1.VCC@2, IC2.IN, IC2.ON/!OFF, IC4.VCC, JTAG.4, R5.2, S5.1, S5.2, S5.3, S5.4, S5.5, S5.6, S5.7, S5.8
- net DGND: now also R17.1, R18.1, U$2.GND, U$3.GND; no longer C13.2, C17.2, C18.2, IC2.GND, IC3A.INH, IC3A.SER, JTAG.10, JTAG.2, R23.2, R24.2, R35.2, R38.2, R39.2, R40.2, R41.2, R43.2
- net GND: now also JP3.2, JP3.4, JTAG.10, JTAG.2, R11.2, UART_ROBO2.1, UART_ROBO2.2, UART_ROBO2.3, V12.S, X1.4, X3-4.S; no longer C10.-, C14.2, C15.2, C16.2, C6.2, LCD1.GND, LCD1.LED-, LCD1.RS(CS), PORT_A.1, PORT_A.10, PORT_D.1, PORT_D.10, R14.1, R16.1, R18.1, R6.2, R7.2, RS232_BT.5, RS232_BT.6, U$1.5, U$1.GND1, U$1.GND2, U$1.GND3, U$1.GND4, U$1.GND5, U$1.GND6, U$1.GND7, U$1.GND8, U$3.GND, UART_ROBO.1, UART_ROBO1.1, V1.S, V2.S, V3.S, V4.S, V5.S, V6.S, V7.S, V8.S, X1-GND.KL, X2-1.SK
- net N$14: now also JP2.3; no longer RS232_BT.2
- net N$15: now also JP2.1; no longer RS232_BT.4
- net N$3: now also IC4.(PCINT11/RESET/DW)PB3, R10.2; no longer F2.1, U$1.1
- net N$5: now also IC4.(PCINT10/INT0/OC0A/CKOUT)PB2, R9.2; no longer H2.C, R26.2
- net N$6: now also IC4.(PCINT9/XTAL2)PB1, R7.2; no longer H1.C, R25.2
- net N$7: now also IC4.(PCINT8/XTAL1/CLKI)PB0, R6.2; no longer R25.1, V1.D
- net PA0: now also R6.1; no longer PORT_A.2, PORT_A2.1
- net PA1: now also R7.1; no longer PORT_A.3, PORT_A2.3
- net PA2: now also R9.1; no longer PORT_A.4, PORT_A2.5
- net PA3: now also R10.1; no longer PORT_A.5, PORT_A2.7
- net PA4: no longer PORT_A.6
- net PA5: no longer IC3A.SH/!LD, PORT_A.7
- net PA6: no longer IC3A.CLK, PORT_A.8
- net PA7: no longer PORT_A.9, R12.2
- net PB0: no longer V8.G
- net PB1: no longer V7.G
- net PB2: no longer R9.2, V6.G
- net PB3: no longer R10.2, V5.G
- net PB4: no longer V4.G
- net PB5: no longer V3.G
- net PB6: no longer V2.G
- net PB7: no longer V1.G
- net PC0: no longer R13.2
- net PC1: no longer R11.2
- net PC6: no longer C16.1, Q2.2
- net PC7: no longer C15.1, Q2.1
- net PD0: now also JP2.2; no longer PORT_D.2, RS232_BT.3
- net PD1: now also JP2.4; no longer PORT_D.3, RS232_BT.1
- net PD2: now also JP1.1; no longer PORT_D.4, UART_ROBO.2
- net PD3: now also JP1.4, PIEZO-POWER1.1; no longer PORT_D.5, UART_ROBO.3
- net PD4: now also JP4.1; no longer PORT_D.6
- net PD5: now also JP4.2; no longer PORT_D.7
- net PD6: now also JP4.3; no longer PORT_D.8
- net PD7: now also JP4.4; no longer PORT_D.9
- net VCC: now also C2.1, C4.1, C7.1, IC1.VCC, IC1.VCC@1, IC1.VCC@2, IC4.VCC, JTAG.4, PIEZO-POWER2.1, R21.1, R5.2, UART_ROBO1.1, UART_ROBO1.2, UART_ROBO1.3; no longer C10.+, C6.1, F2.2, LCD-POWER.1, LED-POWER.1, S3.1, S3.2, S4.1, S4.2, VCC.MP
Other:
- note added: "nc"
- note removed: "8DIP-Switch"
- note removed: "LCD"
- note removed: "LCD 4x20 Zeichen"
- note removed: "LCD-Kontrast"
- note removed: "LED's"
- note removed: "RX"
- note removed: "Spannungsversorgung 5.0V ==> 3.3V"
- note removed: "Spannungsversorgung Mikro-USB 5V ==> 5V"
- note removed: "TX"
- moved on the sheet: +5V-POWER, IC4, PORT_A1, R10, R11, R18, R6, R7, R8, R9

Commit message: sf
Parts:
- removed J1: (no value), con-jack:JACK-PLUG0
- added U$1: BUCHSE, untitled:BUCHSE
Connections:
- net +12V: now also U$1.3, U$1.3.1; no longer J1.3
- net +5V: now also UART_ROBO1.1, UART_ROBO1.2, UART_ROBO1.3
- net DGND: now also JP3.2, JP3.4, U$1.1, U$1.2, UART_ROBO2.1, UART_ROBO2.2, UART_ROBO2.3, X1.4; no longer IC4.GND
- net GND: now also IC4.GND; no longer J1.1, J1.2, JP3.2, JP3.4, UART_ROBO2.1, UART_ROBO2.2, UART_ROBO2.3, X1.4
- net VCC: no longer UART_ROBO1.1, UART_ROBO1.2, UART_ROBO1.3
Other:
- note removed: "Messpunkte"
- moved on the sheet: IC4, JP1, JP3, JTAG, PIEZO-POWER1, PIEZO-POWER2, R10, R11, R18, R21, R6, R7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
