File: Print/Vorlage ATmega644PA.sch (EAGLE design)
At the start: 59 parts, among them IC1 ATmega644PA, IC4 ATTINY24/44/84-SSU, Q1 16MHz, X2 87758-0616

Commit message: asd
Parts:
- removed GND: 3.3V, solpad:LSP11
- removed PIEZO-POWER6: (no value), jumper:JP1E
- removed X2: 87758-0616, con-molex:87758-0616
- added JP2: (no value), jumper:JP3Q
- added R12, R13: 1k, rcl:R-EU_R0805
- added RX, TX: Gruen, led:LEDCHIPLED_1206
- added V1, V2: PMV20EN, transistor-fet-mit-BSS138:BSS138
Connections:
- new net N$2: TX.C, V2.D
- new net N$3: RX.C, V1.D
- new net N$4: R13.1, TX.A
- new net N$5: R12.1, RX.A
- net GND: now also JP2.1, U$4.31, V1.S, V2.S; no longer GND.MP, X2-6.S
- net PA4_: now also JP2.4; no longer X2-3.S
- net PA5_: now also JP2.6; no longer X2-1.S
- net PA6_: now also JP2.3; no longer X2-4.S
- net PB3_: now also JP2.2; no longer X2-5.S
- net PD0: no longer PIEZO-POWER6.2
- net PD1: now also V2.G; no longer PIEZO-POWER6.1
- net PD3: now also V1.G
- net RX: now also U$4.18; no longer U$4.17
- net TX: now also U$4.19; no longer U$4.20
- net VCC: now also JP2.5, R12.2, R13.2; no longer X2-2.S
Other:
- moved on the sheet: U$4
