File: Print/uArm_back_print.sch (EAGLE design)
At the start: 63 parts, among them IC1 ATmega644PA, IC4 ATTINY24/44/84-SSU, Q1 16MHz

Commit message: asd
Parts:
- removed TX: Gruen, led:LEDCHIPLED_1206
- added R14, R15, R16, R19, R20: 1k, rcl:R-EU_R0805
- added RX2, TX1, TX2, TX3, TX4, TX5: Gruen, led:LEDCHIPLED_1206
- added V3, V4: PMV20EN, transistor-fet-mit-BSS138:BSS138
- renumbered RX to RX1
Connections:
- new net N$10: R15.1, RX2.A
- new net N$11: R14.1, TX2.A
- new net N$12: TX2.C, V3.D
- new net N$13: R20.2, TX3.A
- new net N$6: R16.2, TX5.A
- new net N$7: R19.2, TX4.A
- new net N$8: RX2.C, V4.D
- net GND: now also TX3.C, TX4.C, TX5.C, V3.S, V4.S
- net N$2: now also TX1.C; no longer TX.C
- net N$4: now also TX1.A; no longer TX.A
- net PA5: now also R20.1
- net PA6: now also R19.1
- net PA7: now also R16.1
- net PD0: now also V1.G
- net PD2: now also V3.G
- net PD3: now also V4.G; no longer V1.G
- net TX: now also U$4.15; no longer U$4.19
- net VCC: now also R14.2, R15.2
Other:
- note removed: "SRG Clk"
- note removed: "SRG Data"
- note removed: "SRG Load"
- moved on the sheet: R13, V2

Commit message: geschmeus
Parts:
- added 3.3V: 3.3V, solpad:LSP11
- added C10: 1uF, rcl:C-EUC0805
- added C13: 100uF, rcl2:CPOL-EUUD-6,3X8,8
- added C6: 100nF, rcl:C-EUC0805
- added IC2: LP2985-XXDBVR, SmartPrj:LP2985-XXDBVR
- added LSP1, LSP2, LSP3, LSP4, LSP5: LSP11, solpad:LSP11
- added PIEZO-POWER10, PIEZO-POWER8, PIEZO-POWER9: (no value), jumper:JP1E
- added R22, R23, R24: 1k, rcl:R-EU_R0805
- added R25, R26: 1k472, rcl:R-EU_R0805
- added R27: (no value), pot:TRIM_EU-3223G
- C11: value 100nF -> 18pF
- C12: value 100uF -> 18pF; device rcl2:CPOL-EUUD-6,3X8,8 -> rcl:C-EUC0805
- C3, C5: value 18pF -> 100nF
- C9: value 100nF -> 1uF
- R1, R2: value 1k -> 100k
- R11, R21: device rcl:R-EU_R1206 -> rcl:R-EU_R0805
- R17, R18: value 1k472 -> 1k
- R3, R4: value 100k -> 1k
- R5: value 10k -> 1k
Connections:
- new net 3.3V: 3.3V.MP, C9.1, IC2.OUT, R27.E, R27.S
- new net N$14: PIEZO-POWER10.2, R18.1, R22.2
- new net N$15: PIEZO-POWER10.1, R17.1, R23.2
- new net N$17: LSP5.MP, R27.A
- new net N$18: LSP1.MP, R24.1
- new net N$70: C5.1, IC2.NC/FB
- net DGND: now also R25.1, R26.1; no longer R17.1, R18.1
- net GND: now also C10.2, C11.1, C12.2, C13.-, C3.2, C6.1, C9.2, IC2.GND, LSP2.MP, LSP3.MP, LSP4.MP, R1.1, R17.2, R18.2, R2.1; no longer C11.2, C12.-, C3.1, C9.1, R3.1, R4.1
- net N$16: now also R26.2; no longer R18.2
- net N$36: now also C12.1; no longer C5.1
- net N$37: now also C11.2; no longer C3.2
- net N$38: now also C6.2; no longer C9.2
- net N$85: now also R25.2; no longer R17.2
- net PB0: now also R3.1; no longer R1.1
- net PB1: now also R4.1; no longer R2.1
- net PB4: now also PIEZO-POWER9.1
- net PB5: now also PIEZO-POWER9.2
- net PB6: now also PIEZO-POWER8.1
- net PB7: now also PIEZO-POWER8.2
- net PC0: now also R23.1
- net PC1: now also R22.1
- net VCC: now also C10.1, C13.+, C3.1, IC2.IN, IC2.ON/!OFF, R24.2; no longer C11.1, C12.+
Other:
- note added: "Spannungsversorgung 5.0V ==> 3.3V"
- note removed: "Akkuspannung"
- moved on the sheet: C11, C3, C5, C9, R1, R17, R18, R2, R3, R4

Commit message: lol
Parts:
- removed 0_OHM_A: 0 Ohm, rcl:R-EU_R0805
- removed 3.3V: 3.3V, solpad:LSP11
- removed 5V_DC: RECOM_DCDC, DCDC:RECOM_DCDC
- removed D1, D2: MBRS130LT3, diode:MBRS130LT3
- removed LSP1, LSP2, LSP3, LSP4, LSP5: LSP11, solpad:LSP11
- removed PIEZO-POWER1, PIEZO-POWER10, PIEZO-POWER2, PIEZO-POWER3, PIEZO-POWER4, PIEZO-POWER5, PIEZO-POWER8, PIEZO-POWER9: (no value), jumper:JP1E
- removed R27: (no value), pot:TRIM_EU-3223G
- removed TX3, TX4, TX5: Gruen, led:LEDCHIPLED_1206
- removed U$2: DCDC, untitled:DCDC
- removed UART_ROBO1, UART_ROBO2: (no value), jumper:JP2E
- removed V12: PMV20EN, transistor-fet-mit-BSS138:BSS138
- added H1, H2, H3, H4, H5, H6, H7, H8: Gruen, led:LEDCHIPLED_1206
- added JP4, JP5, JP8, JP9: (no value), jumper:JP1E
- added JP6, JP7: (no value), jumper:JP2E
- added LS: ALS-PT17, Lichtsensor:ALS-PT17-51C
- added LS_POTI: 25k, pot:TRIM_EU-3223G
- C11: value 18pF -> 1uF
- C13: value 100uF -> 18pF; device rcl2:CPOL-EUUD-6,3X8,8 -> rcl:C-EUC0805
- C6, C7, C8: value 100nF -> 1uF
- IC2: value LP2985-XXDBVR -> ATTINY24/44/84-SSU; device SmartPrj:LP2985-XXDBVR -> attiny24_44_84:ATTINY24/44/84-SSU
- IC4: value ATTINY24/44/84-SSU -> DCDC; device attiny24_44_84:ATTINY24/44/84-SSU -> untitled:DCDC
- JP2: device jumper:JP3Q -> jumper:JP2Q
- JP3: device jumper:JP2Q -> jumper:JP3Q
- R1, R2: value 100k -> 1k
- R10, R6, R7, R9: value 150R -> 1k
- R23, R24: value 1k -> 1k472
- R25: value 1k472 -> 10k
- R26: value 1k472 -> 100k
- renumbered +5V-POWER to H13, RX1 to H9, RX2 to H12, TX1 to H10, TX2 to H11, U$3 to IC3
Connections:
- removed net 3.3V: 3.3V.MP, C9.1, IC2.OUT, R27.E, R27.S
- removed net N$13: R20.2, TX3.A
- removed net N$46: PIEZO-POWER2.2, R21.2, V12.D
- removed net N$70: C5.1, IC2.NC/FB
- removed net N$75: 5V_DC.IN, C8.1, D1.C, D2.C
- removed net PD8: PIEZO-POWER1.2, R11.1, V12.G
- new net N$19: H6.A, R19.1
- new net N$20: H7.A, R20.1
- new net N$23: H8.A, R21.1
- net +12V: now also IC4.VIN, JP2.1, JP2.3; no longer F1.1, JP3.1, JP3.3, U$2.VIN
- net +5V: now also IC4.VOUT, JP6.1, JP6.2, JP6.3; no longer 0_OHM_A.2, U$2.VOUT, UART_ROBO1.1, UART_ROBO1.2, UART_ROBO1.3
- net DGND: now also IC4.GND, JP2.2, JP2.4, JP7.1, JP7.2, JP7.3, R23.1, R24.1; no longer IC1.GND, IC1.GND@1, IC1.GND@2, IC1.GND@3, JP3.2, JP3.4, R25.1, R26.1, U$2.GND, UART_ROBO2.1, UART_ROBO2.2, UART_ROBO2.3
- net GND: now also C10.1, C13.1, C5.1, C7.1, C8.1, C9.1, H1.C, H2.C, H3.C, H4.C, H5.C, H6.C, H7.C, H8.C, IC1.GND, IC1.GND@1, IC1.GND@2, IC1.GND@3, JP3.1, R25.1; no longer 5V_DC.GND, C10.2, C13.-, C5.2, C7.2, C8.2, C9.2, IC4.GND, JP2.1, LSP2.MP, LSP3.MP, LSP4.MP, R11.2, R17.2, R18.2, TX3.C, TX4.C, TX5.C, V12.S
- net N$1: now also F1.1; no longer PIEZO-POWER4.2
- net N$10: now also R13.1; no longer R15.1
- net N$11: now also R12.1; no longer R14.1
- net N$14: now also H2.A, R15.1; no longer PIEZO-POWER10.2, R18.1, R22.2
- net N$15: now also H3.A, R16.1; no longer PIEZO-POWER10.1, R17.1, R23.2
- net N$16: now also R23.2; no longer R26.2
- net N$17: now also H4.A, R17.1; no longer LSP5.MP, R27.A
- net N$18: now also H5.A, R18.1; no longer LSP1.MP, R24.1
- net N$37: now also C13.2; no longer C11.2
- net N$38: now also C5.2; no longer C6.2
- net N$4: now also R11.1; no longer R13.1
- net N$5: now also R10.1; no longer R12.1
- net N$6: now also LS.E, LS_POTI.A, R26.2; no longer R16.2, TX5.A
- net N$60: now also R22.1; no longer R8.1
- net N$7: now also LS_POTI.E, LS_POTI.S, R25.2; no longer R19.2, TX4.A
- net N$85: now also IC4.TRIM, R24.2; no longer R25.2, U$2.TRIM
- net N$9: now also H1.A, R14.1; no longer D1.A, F1.2
- net PA0_: now also IC2.(PCINT0/AREF/ADC0)PA0; no longer IC4.(PCINT0/AREF/ADC0)PA0
- net PA1_: now also IC2.(PCINT1/AIN0/ADC1)PA1; no longer IC4.(PCINT1/AIN0/ADC1)PA1
- net PA2: now also R8.1; no longer R9.1
- net PA2_: now also IC2.(PCINT2/AIN1/ADC2)PA2; no longer IC4.(PCINT2/AIN1/ADC2)PA2
- net PA3: now also R9.1; no longer R10.1
- net PA3_: now also IC2.(PCINT3/T0/ADC3)PA3; no longer IC4.(PCINT3/T0/ADC3)PA3
- net PA4: now also JP9.2
- net PA4_: now also IC2.(PCINT4/T1/SCL/USCK/ADC4)PA4, JP3.4; no longer IC4.(PCINT4/T1/SCL/USCK/ADC4)PA4, JP2.4
- net PA5: now also JP9.1; no longer R20.1
- net PA5_: now also IC2.(PCINT5/OC1B/MISO/DO/ADC5)PA5, JP3.6; no longer IC4.(PCINT5/OC1B/MISO/DO/ADC5)PA5, JP2.6
- net PA6: now also JP8.2; no longer R19.1
- net PA6_: now also IC2.(PCINT6/OC1A/SDA/MOSI/ADC6)PA6, JP3.3; no longer IC4.(PCINT6/OC1A/SDA/MOSI/ADC6)PA6, JP2.3
- net PA7: now also C11.2, JP8.1, R26.1; no longer R16.1
- net PA7_: now also IC2.(PCINT7/ICP/OC0B/ADC7)PA7; no longer IC4.(PCINT7/ICP/OC0B/ADC7)PA7
- net PB0: now also R14.2; no longer R3.1
- net PB0_: now also IC2.(PCINT8/XTAL1/CLKI)PB0; no longer IC4.(PCINT8/XTAL1/CLKI)PB0
- net PB1: now also R15.2; no longer R4.1
- net PB1_: now also IC2.(PCINT9/XTAL2)PB1; no longer IC4.(PCINT9/XTAL2)PB1
- net PB2: now also R16.2
- net PB2_: now also IC2.(PCINT10/INT0/OC0A/CKOUT)PB2, R8.2; no longer IC4.(PCINT10/INT0/OC0A/CKOUT)PB2, R9.2
- net PB3: now also R17.2
- net PB3_: now also IC2.(PCINT11/RESET/DW)PB3, JP3.2, R9.2; no longer IC4.(PCINT11/RESET/DW)PB3, JP2.2, R10.2
- net PB4: now also R18.2; no longer PIEZO-POWER9.1
- net PB5: now also R19.2; no longer PIEZO-POWER9.2
- net PB6: now also R20.2; no longer PIEZO-POWER8.1
- net PB7: now also R21.2; no longer PIEZO-POWER8.2
- net PC0: no longer R23.1
- net PC1: no longer R22.1
- net PC6: now also R4.1
- net PC7: now also R3.1
- net PD3: no longer PIEZO-POWER1.1
- net PD4: now also JP4.2; no longer PIEZO-POWER3.1
- net PD5: now also JP4.1; no longer PIEZO-POWER5.2
- net PD6: now also JP5.2; no longer PIEZO-POWER3.2
- net PD7: now also JP5.1; no longer PIEZO-POWER5.1
- net VCC: now also C10.2, C6.2, C7.2, C8.2, C9.2, F1.2, IC2.VCC, JP3.5, LS.C, R10.2, R11.2, R22.2; no longer 0_OHM_A.1, 5V_DC.OUT, C10.1, C13.+, C7.1, D2.A, IC2.IN, IC2.ON/!OFF, IC4.VCC, JP2.5, PIEZO-POWER2.1, PIEZO-POWER4.1, R14.2, R15.2, R21.1, R24.2, R8.2
Other:
- note added: "Lichtsensor"
- note removed: "Eingangs-Spannung 6.5V - 36V"
- note removed: "Spannungsversorgung 5.0V ==> 3.3V"
- note removed: "Spannungsversorgung 6.5V-36V ==> 5V"
- note removed: "Taste 1"
- note removed: "Taste 2"
- note removed: "Taste 3"
- note removed: "Taste 4"
- moved on the sheet: 0_OHM_B, C1, C10, C11, C3, C4, C5, C6, C7, C8, C9, F1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

Commit message: yeees
Other:
- moved on the sheet: C10, C6, C7, C8, C9, JP1
