File: Print/TestPrint/TestPrint.brd (EAGLE design)
At the start: 126.8 x 100.1 mm, 65 parts

Commit message: Dinge Geändert
Parts:
- added U$66: TQFP-64, IC-packages_BIG-pack V1.0:TQFP64
- added U$67, U$68: TSSOP24, IC-packages_BIG-pack V1.0:TSSOP24
- U$62: value TQPF-100 -> TQFP-64; device IC-packages_BIG-pack V1.0:TQFP100 -> IC-packages_BIG-pack V1.0:TQFP64
- moved U$62 11.9 mm to (36.0, 81.0), turned to 0 degrees
- moved U$63 5.49 mm to (38.7, 25.6)
- moved U$61 4.59 mm to (14.9, 24.9)
- moved U$54 3.66 mm to (117.3, 70.5)
- moved U$55 3.35 mm to (55.1, 68.6)
- moved U$53 2.34 mm to (105.8, 70.5)
- moved U$58 2.03 mm to (54.5, 84.5)
- moved U$52 1.32 mm to (94.7, 70.5)
- moved U$60 0.91 mm to (36.4, 60.3)
Other:
- board text added: "LQFP-48"
- board text added: "TQFP-64"
Changed lines of the file:
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@@
 <wire x1="123.19" y1="50.8" x2="123.19" y2="58.42" width="0.1524" layer="25"/>
 <wire x1="76.835" y1="64.135" x2="76.835" y2="76.835" width="0.1524" layer="25"/>
-<wire x1="76.835" y1="76.835" x2="118.745" y2="76.835" width="0.1524" layer="25"/>
-<wire x1="118.745" y1="76.835" x2="118.745" y2="64.135" width="0.1524" layer="25"/>
-<wire x1="118.745" y1="64.135" x2="76.835" y2="64.135" width="0.1524" layer="25"/>
-<wire x1="51.435" y1="79.375" x2="51.435" y2="90.805" width="0.1524" layer="25"/>
-<wire x1="51.435" y1="90.805" x2="70.485" y2="90.805" width="0.1524" layer="25"/>
-<wire x1="70.485" y1="90.805" x2="70.485" y2="79.375" width="0.1524" layer="25"/>
-<wire x1="70.485" y1="79.375" x2="51.435" y2="79.375" width="0.1524" layer="25"/>
+<wire x1="76.835" y1="76.835" x2="123.4186" y2="77.1398" width="0.1524" layer="25"/>
+<wire x1="123.4186" y1="77.1398" x2="123.4186" y2="64.4398" width="0.1524" layer="25"/>
+<wire x1="123.4186" y1="64.4398" x2="76.835" y2="64.135" width="0.1524" layer="25"/>
+<wire x1="48.4886" y1="79.375" x2="48.4886" y2="90.805" width="0.1524" layer="25"/>
+<wire x1="48.4886" y1="90.805" x2="99.1362" y2="90.805" width="0.1524" layer="25"/>
+<wire x1="99.1362" y1="90.805" x2="99.1362" y2="79.375" width="0.1524" layer="25"/>
+<wire x1="99.1362" y1="79.375" x2="48.4886" y2="79.375" width="0.1524" layer="25"/>
 <text x="57.15" y="15.875" size="1.778" layer="25">0402</text>
 <text x="56.896" y="24.384" size="1.778" layer="25">0603</text>
@@
 <text x="76.9112" y="61.8236" size="1.778" layer="25">SO-14</text>
 <text x="51.435" y="91.44" size="1.778" layer="25">TSSOP-24</text>
-<wire x1="53.34" y1="64.77" x2="53.34" y2="72.39" width="0.1524" layer="25"/>
-<wire x1="53.34" y1="72.39" x2="70.485" y2="72.39" width="0.1524" layer="25"/>
+<wire x1="49.9872" y1="64.77" x2="49.9872" y2="72.39" width="0.1524" layer="25"/>
+<wire x1="49.9872" y1="72.39" x2="70.485" y2="72.39" width="0.1524" layer="25"/>
 <wire x1="70.485" y1="72.39" x2="70.485" y2="64.77" width="0.1524" layer="25"/>
-<wire x1="70.485" y1="64.77" x2="53.34" y2="64.77" width="0.1524" layer="25"/>
+<wire x1="70.485" y1="64.77" x2="49.9872" y2="64.77" width="0.1524" layer="25"/>
 <text x="52.705" y="73.025" size="1.778" layer="25">TSSOP-14</text>
+<wire x1="4.1656" y1="17.272" x2="4.1656" y2="47.752" width="0.1524" layer="25"/>
+<wire x1="4.1656" y1="47.752" x2="45.4152" y2="47.752" width="0.1524" layer="25"/>
+<wire x1="45.4152" y1="47.752" x2="45.4152" y2="16.9672" width="0.1524" layer="25"/>
+<wire x1="45.4152" y1="16.9672" x2="3.9624" y2="16.9672" width="0.1524" layer="25"/>
+<wire x1="3.8608" y1="93.3704" x2="3.8608" y2="48.768" width="0.1524" layer="25"/>
+<wire x1="3.8608" y1="48.768" x2="45.6184" y2="48.768" width="0.1524" layer="25"/>
+<wire x1="45.6184" y1="48.768" x2="45.6184" y2="93.1672" width="0.1524" layer="25"/>
+<wire x1="45.6184" y1="93.1672" x2="3.9624" y2="93.1672" width="0.1524" layer="25"/>
+<text x="4.3688" y="13.8176" size="1.778" layer="25">LQFP-48</text>
+<text x="3.9624" y="93.3704" size="1.778" layer="25">TQFP-64</text>
 </plain>
 <attributes>
@@
 <element name="U$50" library="IC-packages_BIG-pack V1.0" package="SOT23" value="SOTSOT-23" x="119.38" y="54.61" smashed="yes" rot="R180"/>
 <element name="U$51" library="IC-packages_BIG-pack V1.0" package="SO14" value="SO14SO14" x="83.185" y="70.485" smashed="yes" rot="R90"/>
-<element name="U$52" library="IC-packages_BIG-pack V1.0" package="SO14" value="SO14SO14" x="93.345" y="70.485" smashed="yes" rot="R90"/>
-<element name="U$53" library="IC-packages_BIG-pack V1.0" package="SO14" value="SO14SO14" x="103.505" y="70.485" smashed="yes" rot="R90"/>
-<element name="U$54" library="IC-packages_BIG-pack V1.0" package="SO14" value="SO14SO14" x="113.665" y="70.485" smashed="yes" rot="R90"/>
-<element name="U$55" library="IC-packages_BIG-pack V1.0" package="TSSOP14" value="TSSOP14" x="58.42" y="68.58" smashed="yes" rot="R90"/>
+<element name="U$52" library="IC-packages_BIG-pack V1.0" package="SO14" value="SO14SO14" x="94.6658" y="70.485" smashed="yes" rot="R90"/>
+<element name="U$53" library="IC-packages_BIG-pack V1.0" package="SO14" value="SO14SO14" x="105.8418" y="70.485" smashed="yes" rot="R90"/>
+<element name="U$54" library="IC-packages_BIG-pack V1.0" package="SO14" value="SO14SO14" x="117.3226" y="70.485" smashed="yes" rot="R90"/>
+<element name="U$55" library="IC-packages_BIG-pack V1.0" package="TSSOP14" value="TSSOP14" x="55.0672" y="68.58" smashed="yes" rot="R90"/>
 <element name="U$56" library="IC-packages_BIG-pack V1.0" package="TSSOP14" value="TSSOP14" x="66.04" y="68.58" smashed="yes" rot="R90"/>
-<element name="U$58" library="IC-packages_BIG-pack V1.0" package="TSSOP24" value="TSSOP24" x="56.515" y="84.455" smashed="yes" rot="R90"/>
+<element name="U$58" library="IC-packages_BIG-pack V1.0" package="TSSOP24" value="TSSOP24" x="54.483" y="84.455" smashed="yes" rot="R90"/>
 <element name="U$59" library="IC-packages_BIG-pack V1.0" package="TSSOP24" value="TSSOP24" x="65.405" y="84.455" smashed="yes" rot="R90"/>
-<element name="U$60" library="IC-packages_BIG-pack V1.0" package="TQFP64" value="TQFP-64" x="37.338" y="60.2996" smashed="yes" rot="R90">
-<attribute name="VALUE" x="33.909" y="59.0423" size="1.27" layer="27"/>
-</element>
-<element name="U$61" library="IC-packages_BIG-pack V1.0" package="LQFP48" value="LQFP-48" x="15.3416" y="20.32" smashed="yes" rot="R90">
-<attribute name="VALUE" x="11.1506" y="26.035" size="1.27" layer="27"/>
-</element>
-<element name="U$62" library="IC-packages_BIG-pack V1.0" package="TQFP100" value="TQPF-100" x="24.7904" y="85.09" smashed="yes" rot="R90">
-<attribute name="VALUE" x="19.0754" y="84.455" size="1.778" layer="27" ratio="10"/>
-</element>
+<element name="U$60" library="IC-packages_BIG-pack V1.0" package="TQFP64" value="TQFP-64" x="36.4236" y="60.2996" smashed="yes" rot="R90"/>
+<element name="U$61" library="IC-packages_BIG-pack V1.0" package="LQFP48" value="LQFP-48" x="14.9352" y="24.892" smashed="yes" rot="R90"/>
 <element name="U$64" library="IC-packages_BIG-pack V1.0" package="TQFP64" value="TQFP-64" x="14.0208" y="60.2488" smashed="yes">
 <attribute name="NAME" x="7.9248" y="68.7705" size="1.27" layer="25"/>
-<attribute name="VALUE" x="7.6708" y="58.3565" size="1.27" layer="27"/>
-</element>
-<element name="U$65" library="IC-packages_BIG-pack V1.0" package="LQFP48" value="LQFP-48" x="14.8336" y="40.0304" smashed="yes">
-<attribute name="VALUE" x="10.9728" y="45.7708" size="1.27" layer="27"/>
-</element>
-<element name="U$57" library="IC-packages_BIG-pack V1.0" package="LQFP48" value="LQFP-48" x="38.3032" y="39.7256" smashed="yes">
-<attribute name="VALUE" x="34.7472" y="45.2628" size="1.27" layer="27"/>
-</element>
-<element name="U$63" library="IC-packages_BIG-pack V1.0" package="LQFP48" value="LQFP-48" x="38.7096" y="20.1168" smashed="yes">
-<attribute name="VALUE" x="35.1536" y="25.9588" size="1.27" layer="27"/>
+</element>
+<element name="U$65" library="IC-packages_BIG-pack V1.0" package="LQFP48" value="LQFP-48" x="14.8336" y="40.0304" smashed="yes"/>
+<element name="U$57" library="IC-packages_BIG-pack V1.0" package="LQFP48" value="LQFP-48" x="38.3032" y="39.7256" smashed="yes"/>
+<element name="U$63" library="IC-packages_BIG-pack V1.0" package="LQFP48" value="LQFP-48" x="38.7096" y="25.6032" smashed="yes"/>
+<element name="U$62" library="IC-packages_BIG-pack V1.0" package="TQFP64" value="TQFP-64" x="35.9664" y="80.9752" smashed="yes">
+<attribute name="NAME" x="29.8704" y="89.4969" size="1.27" layer="25"/>
+</element>
+<element name="U$66" library="IC-packages_BIG-pack V1.0" package="TQFP64" value="TQFP-64" x="14.3256" y="81.28" smashed="yes">
+<attribute name="NAME" x="8.2296" y="89.8017" size="1.27" layer="25"/>
+</element>
+<element name="U$67" library="IC-packages_BIG-pack V1.0" package="TSSOP24" value="TSSOP24" x="77.5208" y="84.328" smashed="yes" rot="R90">
+<attribute name="NAME" x="79.6036" y="80.1324" size="1.016" layer="25" ratio="10" rot="R180"/>
+<attribute name="VALUE" x="79.6036" y="89.5142" size="1.016" layer="27" ratio="10" rot="R180"/>
+</element>
+<element name="U$68" library="IC-packages_BIG-pack V1.0" package="TSSOP24" value="TSSOP24" x="88.7984" y="84.2264" smashed="yes" rot="R90">
+<attribute name="NAME" x="90.8812" y="80.0308" size="1.016" layer="25" ratio="10" rot="R180"/>
+<attribute name="VALUE" x="90.8812" y="89.4126" size="1.016" layer="27" ratio="10" rot="R180"/>
 </element>
 </elements>
