File: Print/TestPrint/TestPrint.sch (EAGLE design)
At the start: 65 parts

Commit message: Dinge Geändert
Parts:
- added U$66: TQFP-64, IC-packages_BIG-pack V1.0:TQFP-64
- added U$67, U$68: TSSOP24, IC-packages_BIG-pack V1.0:TSSOP24
- U$62: value TQPF-100 -> TQFP-64; device IC-packages_BIG-pack V1.0:TQPF-100 -> IC-packages_BIG-pack V1.0:TQFP-64
Changed lines of the file:
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@@
 <part name="U$60" library="IC-packages_BIG-pack V1.0" deviceset="TQFP-64" device=""/>
 <part name="U$61" library="IC-packages_BIG-pack V1.0" deviceset="LQFP-48" device=""/>
-<part name="U$62" library="IC-packages_BIG-pack V1.0" deviceset="TQPF-100" device=""/>
 <part name="U$64" library="IC-packages_BIG-pack V1.0" deviceset="TQFP-64" device=""/>
 <part name="U$65" library="IC-packages_BIG-pack V1.0" deviceset="LQFP-48" device=""/>
 <part name="U$57" library="IC-packages_BIG-pack V1.0" deviceset="LQFP-48" device=""/>
 <part name="U$63" library="IC-packages_BIG-pack V1.0" deviceset="LQFP-48" device=""/>
+<part name="U$62" library="IC-packages_BIG-pack V1.0" deviceset="TQFP-64" device=""/>
+<part name="U$66" library="IC-packages_BIG-pack V1.0" deviceset="TQFP-64" device=""/>
+<part name="U$67" library="IC-packages_BIG-pack V1.0" deviceset="TSSOP24" device=""/>
+<part name="U$68" library="IC-packages_BIG-pack V1.0" deviceset="TSSOP24" device=""/>
 </parts>
 <sheets>
@@
 <instance part="U$60" gate="G$1" x="-167.64" y="264.16" smashed="yes"/>
 <instance part="U$61" gate="G$1" x="-182.88" y="264.16" smashed="yes"/>
-<instance part="U$62" gate="G$1" x="-160.02" y="264.16" smashed="yes"/>
 <instance part="U$64" gate="G$1" x="-167.64" y="256.54" smashed="yes"/>
 <instance part="U$65" gate="G$1" x="-182.88" y="256.54" smashed="yes"/>
 <instance part="U$57" gate="G$1" x="-182.88" y="248.92" smashed="yes"/>
 <instance part="U$63" gate="G$1" x="-182.88" y="241.3" smashed="yes"/>
+<instance part="U$62" gate="G$1" x="-167.64" y="248.92" smashed="yes"/>
+<instance part="U$66" gate="G$1" x="-167.64" y="241.3" smashed="yes"/>
+<instance part="U$67" gate="G$1" x="-195.58" y="248.92" smashed="yes"/>
+<instance part="U$68" gate="G$1" x="-195.58" y="241.3" smashed="yes"/>
 </instances>
 <busses>
