File: Print/V3.0/uArm_back_print.sch (EAGLE design)
At the start: 82 parts, among them IC1 ATmega644PA, IC2 ATTINY24/44/84-SSU, IC3 DCDC, IC4 DCDC, Q1 16MHz

Commit message: lol
Parts:
- removed H1, H2, H3, H4, H5, H6, H7, H8: Gruen, led:LEDCHIPLED_1206
- removed LS: ALS-PT17, Lichtsensor:ALS-PT17-51C
- removed LS_POTI: 25k, pot:TRIM_EU-3223G
- added 0_OHM_A: 0 Ohm, rcl:R-EU_R0805
- added 3.3V: 3.3V, solpad:LSP11
- added 5V_DC: RECOM_DCDC, DCDC:RECOM_DCDC
- added D1, D2: MBRS130LT3, diode:MBRS130LT3
- added LSP1, LSP2, LSP3, LSP4, LSP5: LSP11, solpad:LSP11
- added PIEZO-POWER1, PIEZO-POWER10, PIEZO-POWER2, PIEZO-POWER4, PIEZO-POWER8, PIEZO-POWER9: (no value), jumper:JP1E
- added R27: (no value), pot:TRIM_EU-3223G
- added TX3, TX4, TX5: Gruen, led:LEDCHIPLED_1206
- added U$2: DCDC, untitled:DCDC
- added V12: PMV20EN, transistor-fet-mit-BSS138:BSS138
- C10, C9: device rcl:C-EUC0603 -> rcl:C-EUC0805
- C11: value 1uF -> 18pF; device rcl:C-EUC0603 -> rcl:C-EUC0805
- C13: value 18pF -> 100uF; device rcl:C-EUC0805 -> rcl2:CPOL-EUUD-6,3X8,8
- C6, C7, C8: value 1uF -> 100nF; device rcl:C-EUC0603 -> rcl:C-EUC0805
- IC2: value ATTINY24/44/84-SSU -> LP2985-XXDBVR; device attiny24_44_84:ATTINY24/44/84-SSU -> SmartPrj:LP2985-XXDBVR
- IC4: value DCDC -> ATTINY24/44/84-SSU; device untitled:DCDC -> attiny24_44_84:ATTINY24/44/84-SSU
- R1, R2: value 1k -> 100k
- R10, R6, R7, R9: value 1k -> 150R
- R23, R24: value 1k472 -> 1k
- R25: value 10k -> 1k472
- R26: value 100k -> 1k472
- renumbered IC3 to U$3
Connections:
- removed net N$19: H6.A, R19.1
- removed net N$20: H7.A, R20.1
- removed net N$23: H8.A, R21.1
- new net 3.3V: 3.3V.MP, C9.1, IC2.OUT, R27.E, R27.S
- new net N$13: R20.2, TX3.A
- new net N$46: PIEZO-POWER2.2, R21.2, V12.D
- new net N$70: C5.1, IC2.NC/FB
- new net N$75: 5V_DC.IN, C8.1, D1.C, D2.C
- new net PD8: PIEZO-POWER1.2, R11.1, V12.G
- net +12V: now also F1.1, U$2.VIN; no longer IC4.VIN
- net +5V: now also 0_OHM_A.2, U$2.VOUT; no longer IC4.VOUT
- net DGND: now also IC1.GND, IC1.GND@1, IC1.GND@2, IC1.GND@3, R25.1, R26.1, U$2.GND; no longer IC4.GND, R23.1, R24.1
- net GND: now also 5V_DC.GND, C10.2, C13.-, C5.2, C7.2, C8.2, C9.2, IC4.GND, LSP2.MP, LSP3.MP, LSP4.MP, R11.2, R17.2, R18.2, TX3.C, TX4.C, TX5.C, V12.S; no longer C10.1, C13.1, C5.1, C7.1, C8.1, C9.1, H1.C, H2.C, H3.C, H4.C, H5.C, H6.C, H7.C, H8.C, IC1.GND, IC1.GND@1, IC1.GND@2, IC1.GND@3, R25.1
- net N$1: now also PIEZO-POWER4.2; no longer F1.1
- net N$10: now also R15.1; no longer R13.1
- net N$11: now also R14.1; no longer R12.1
- net N$14: now also PIEZO-POWER10.2, R18.1, R22.2; no longer H2.A, R15.1
- net N$15: now also PIEZO-POWER10.1, R17.1, R23.2; no longer H3.A, R16.1
- net N$16: now also R26.2; no longer R23.2
- net N$17: now also LSP5.MP, R27.A; no longer H4.A, R17.1
- net N$18: now also LSP1.MP, R24.1; no longer H5.A, R18.1
- net N$37: now also C11.2; no longer C13.2
- net N$38: now also C6.2; no longer C5.2
- net N$4: now also R13.1; no longer R11.1
- net N$5: now also R12.1; no longer R10.1
- net N$6: now also R16.2, TX5.A; no longer LS.E, LS_POTI.A, R26.2
- net N$60: now also R8.1; no longer R22.1
- net N$7: now also R19.2, TX4.A; no longer LS_POTI.E, LS_POTI.S, R25.2
- net N$85: now also R25.2, U$2.TRIM; no longer IC4.TRIM, R24.2
- net N$9: now also D1.A, F1.2; no longer H1.A, R14.1
- net PA0_: now also IC4.(PCINT0/AREF/ADC0)PA0; no longer IC2.(PCINT0/AREF/ADC0)PA0
- net PA1_: now also IC4.(PCINT1/AIN0/ADC1)PA1; no longer IC2.(PCINT1/AIN0/ADC1)PA1
- net PA2: now also R9.1; no longer R8.1
- net PA2_: now also IC4.(PCINT2/AIN1/ADC2)PA2; no longer IC2.(PCINT2/AIN1/ADC2)PA2
- net PA3: now also R10.1; no longer R9.1
- net PA3_: now also IC4.(PCINT3/T0/ADC3)PA3; no longer IC2.(PCINT3/T0/ADC3)PA3
- net PA4_: now also IC4.(PCINT4/T1/SCL/USCK/ADC4)PA4; no longer IC2.(PCINT4/T1/SCL/USCK/ADC4)PA4
- net PA5: now also R20.1
- net PA5_: now also IC4.(PCINT5/OC1B/MISO/DO/ADC5)PA5; no longer IC2.(PCINT5/OC1B/MISO/DO/ADC5)PA5
- net PA6: now also R19.1
- net PA6_: now also IC4.(PCINT6/OC1A/SDA/MOSI/ADC6)PA6; no longer IC2.(PCINT6/OC1A/SDA/MOSI/ADC6)PA6
- net PA7: now also R16.1; no longer C11.2, R26.1
- net PA7_: now also IC4.(PCINT7/ICP/OC0B/ADC7)PA7; no longer IC2.(PCINT7/ICP/OC0B/ADC7)PA7
- net PB0: now also R3.1; no longer R14.2
- net PB0_: now also IC4.(PCINT8/XTAL1/CLKI)PB0; no longer IC2.(PCINT8/XTAL1/CLKI)PB0
- net PB1: now also R4.1; no longer R15.2
- net PB1_: now also IC4.(PCINT9/XTAL2)PB1; no longer IC2.(PCINT9/XTAL2)PB1
- net PB2: no longer R16.2
- net PB2_: now also IC4.(PCINT10/INT0/OC0A/CKOUT)PB2, R9.2; no longer IC2.(PCINT10/INT0/OC0A/CKOUT)PB2, R8.2
- net PB3: no longer R17.2
- net PB3_: now also IC4.(PCINT11/RESET/DW)PB3, R10.2; no longer IC2.(PCINT11/RESET/DW)PB3, R9.2
- net PB4: now also PIEZO-POWER9.1; no longer R18.2
- net PB5: now also PIEZO-POWER9.2; no longer R19.2
- net PB6: now also PIEZO-POWER8.1; no longer R20.2
- net PB7: now also PIEZO-POWER8.2; no longer R21.2
- net PC0: now also R23.1
- net PC1: now also R22.1
- net PC6: no longer R4.1
- net PC7: no longer R3.1
- net PD3: now also PIEZO-POWER1.1
- net PD4: now also PIEZO-POWER3.1; no longer PIEZO-POWER3.2
- net PD5: now also PIEZO-POWER5.2; no longer PIEZO-POWER3.1
- net PD6: now also PIEZO-POWER3.2; no longer PIEZO-POWER5.2
- net VCC: now also 0_OHM_A.1, 5V_DC.OUT, C10.1, C13.+, C7.1, D2.A, IC2.IN, IC2.ON/!OFF, IC4.VCC, PIEZO-POWER2.1, PIEZO-POWER4.1, R14.2, R15.2, R21.1, R24.2, R8.2; no longer C10.2, C6.2, C7.2, C8.2, C9.2, F1.2, IC2.VCC, LS.C, R10.2, R11.2, R22.2
Other:
- note added: "Eingangs-Spannung 6.5V - 36V"
- note added: "Spannungsversorgung 5.0V ==> 3.3V"
- note added: "Spannungsversorgung 6.5V-36V ==> 5V"
- note added: "Taste 1"
- note added: "Taste 2"
- note added: "Taste 3"
- note added: "Taste 4"
- note removed: "Lichtsensor"
- moved on the sheet: 0_OHM_B, C1, C10, C11, C3, C4, C5, C6, C7, C8, C9, F1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
